File: Schematy Połączeń/Schematy/untitled.kicad_sch (KiCad schematic)
At the start: 5 parts, among them Q3 2N2219, U4 ESP32-WROOM-32

Commit message: Dokument do zaliczenia 7 semestru
Connections:
- net at R6.1: now also U4.16 (IO13); no longer U4.29 (IO5)
Changed lines of the file:
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@@
 	(wire
 		(pts
-			(xy 114.3 90.17) (xy 114.3 82.55)
+			(xy 114.3 85.09) (xy 114.3 82.55)
 		)
 		(stroke
@@
 		(pts
 			(xy 59.69 31.75) (xy 73.66 31.75)
-		)
-		(stroke
-			(width 0)
-			(type default)
-		)
-	)
-	(wire
-		(pts
-			(xy 114.3 90.17) (xy 120.65 90.17)
 		)
 		(stroke
@@
 		)
 		(stroke
+			(width 0)
+			(type default)
+		)
+	)
+	(wire
+		(pts
+			(xy 114.3 85.09) (xy 120.65 85.09)
+		)
+		(stroke
